Commit message: Adding Visual Servoing

File: visual_servoing/robot/camera.xacro (robot description, xacro)
@@ -18,5 +18,5 @@
       <material>Gazebo/Yellow</material>
   		<sensor name="camera" type="depth">
-        <update_rate>10</update_rate>
+        <update_rate>30</update_rate>
         <camera>
           <horizontal_fov>1.047198</horizontal_fov>

File: visual_servoing/robot/scara_arm.urdf.xacro (robot description, xacro)
@@ -12,4 +12,5 @@
   <!-- <xacro:camera3D pLink="scara_link3" xyz='0.025 0 0.1' rpy='0 -${PI/2} -${PI/2}' /> -->
   <!-- <xacro:camera3D pLink="scara_link3" xyz='0 0 0.11' rpy='0 -${PI/2} -${PI/2}' /> -->
-  <xacro:camera3D pLink="scara_link2B" xyz='0.04 0 0.03' rpy='${0} -${PI/2+0.269} -${0*PI/2}' />
+  <!-- <xacro:camera3D pLink="scara_link2B" xyz='0.04 0 0.03' rpy='${0} -${PI/2-0.269} -${2*PI/2}' /> -->
+  <xacro:camera3D pLink="scara_link2B" xyz='0.04 0 0.03' rpy='${0} -${PI/2} -${2*PI/2}' />
 </robot>

File: visual_servoing/robot/scara_arm.xacro (robot description, xacro)
@@ -4,5 +4,5 @@
 <robot xmlns:xacro="http://www.ros.org/wiki/xacro" name = "scara">
 	<xacro:include filename="$(find visual_servoing)/robot/links.xacro"/>
-	<xacro:macro name="scara_arm" params="arm_id:='scara' connected_to:='' c_xyz='0 0 0' c_rpy=:='000'">
+	<xacro:macro name="scara_arm" params="arm_id:='scara' connected_to:='' c_xyz='0 0 0' c_rpy=:='0 0 0'">
 		<xacro:unless value="${not connected_to}">
 			<joint name="${arm_id}_joint_${connected_to}" type="fixed">
@@ -52,5 +52,5 @@
 		<!-- Link 3 : Prismatic Joint -->
 		<link name = "${arm_id}_link3">
-			<xacro:linkCylinder density="2710" rad="0.01" len= "0.2" xyz="0 0 0" rpy="0 0 0"/>
+			<xacro:linkCylinder density="${4*2710}" rad="${0.01/2}" len= "0.2" xyz="0 0 0" rpy="0 0 0"/>
 		</link>
 		<gazebo reference="${arm_id}_link3">
@@ -59,5 +59,5 @@
 		<!-- Link 4 : Revolute Joint -->
 		<link name = "${arm_id}_link4">
-			<xacro:linkCylinder density="2710" rad="0.012" len= "0.01" xyz="0 0 -0.005" rpy="0 0 0"/>
+			<xacro:linkCylinder density="${4*2710}" rad="${0.012/2}" len= "0.01" xyz="0 0 -0.005" rpy="0 0 0"/>
 		</link>
 		<gazebo reference="${arm_id}_link4">

File: visual_servoing/robot/tt.urdf.xacro (robot description, xacro)
@@ -29,5 +29,5 @@
 		<child link="${tt_id}_A"/>
 		<origin xyz="0.2 -0.2 0.0" rpy="0 0 0"/>
-		<limit effort="30.0" velocity="${PI/10}"/>
+		<limit effort="30.0" velocity="${PI/5}"/>
 		<axis xyz="0 0 1"/>
 	</joint>
